Commit message: the fucking day comes to an end!

File: mbzirc_task2/ur5_manipulation/urdf/table_ipa.urdf.xacro (robot description, xacro)
@@ -12,5 +12,5 @@
       <origin xyz="0 0 0" rpy="0 0 0.0" />
       <geometry>
-        <mesh filename="package://ur5_collision/meshes/RoboterzelleSmaller.stl" scale="0.001 0.001 0.001" />
+        <mesh filename="package://ur5_manipulation/meshes/RoboterzelleSmaller.stl" scale="0.001 0.001 0.001" />
       </geometry>
       <material name="Grey">

File: mbzirc_task2/ur5_manipulation/urdf/table_scene_gazebo.urdf.xacro (robot description, xacro)
@@ -1,5 +1,5 @@
 <?xml version="1.0"?>
 <robot name="ur5" xmlns:xacro="http://ros.org/wiki/xacro">
-  <xacro:include filename="$(find ur5_collision)/urdf/table_ipa.urdf.xacro" />
+  <xacro:include filename="$(find ur5_manipulation)/urdf/table_ipa.urdf.xacro" />
   <xacro:include filename="$(find ur_description)/urdf/ur5.urdf.xacro" />
   <xacro:include filename="$(find ur_description)/urdf/common.gazebo.xacro" />

File: mbzirc_task2/ur5_manipulation/urdf/table_scene_real_robot.urdf.xacro (robot description, xacro)
@@ -1,5 +1,5 @@
 <?xml version="1.0"?>
 <robot name="ur5" xmlns:xacro="http://ros.org/wiki/xacro">
-  <xacro:include filename="$(find ur5_collision)/urdf/table_ipa.urdf.xacro" />
+  <xacro:include filename="$(find ur5_manipulation)/urdf/table_ipa.urdf.xacro" />
   <xacro:include filename="$(find ur_description)/urdf/ur5.urdf.xacro" />
   <xacro:include filename="$(find ur_description)/urdf/common.gazebo.xacro" />
