Commit message: Converted the wrench pose in UR5 frame (at the moment in world frame) Fairly accurate.. actually off by 10cm!

File: mbzirc_task2/ur5_manipulation/urdf/ur5_robot.urdf.xacro (robot description, xacro)
@@ -4,4 +4,6 @@
   <!-- ur5 -->
   <xacro:include filename="$(find ur_description)/urdf/ur5.urdf.xacro" />
+  <xacro:include filename="$(find sick_tim)/urdf/sick_tim.urdf.xacro" />
+  <xacro:sick_tim310 name="laser" ros_topic="scan" />
   <!-- arm -->
   <xacro:ur5_robot prefix="" joint_limited="false"/>
@@ -10,5 +12,10 @@
     <parent link="world" />
     <child link = "base_link" />
-    <origin xyz="0.0 0.0 0.0" rpy="0.0 0.0 0.0" />
+    <origin xyz="0.0 0.0 0.75" rpy="0.0 0.0 0.0" />
+  </joint>
+  <joint name="tim_link" type="fixed">
+	<parent link="base_link" />
+    <child link = "laser_mount_link" />
+    <origin xyz="-0.28 0 0" rpy="0.0 0.0 3.142" />
   </joint>
 </robot>

Commit message: added functionaliy for wrench pose detection and wrench pick. Tested, works.

File: mbzirc_task2/ur5_manipulation/urdf/ur5_robot.urdf.xacro (robot description, xacro)
@@ -17,5 +17,5 @@
 	<parent link="base_link" />
     <child link = "laser_mount_link" />
-    <origin xyz="-0.28 0 0" rpy="0.0 0.0 3.142" />
+    <origin xyz="-0.28 0.01 0" rpy="0.0 0.0 3.142" />
   </joint>
 </robot>

Commit message: Integration with Husky issues

File: mbzirc_task2/ur5_manipulation/urdf/ur5_robot.urdf.xacro (robot description, xacro)
@@ -3,7 +3,5 @@
        name="ur5" >
   <!-- ur5 -->
-  <xacro:include filename="$(find ur_description)/urdf/ur5.urdf.xacro" />
-  <xacro:include filename="$(find sick_tim)/urdf/sick_tim.urdf.xacro" />
-  <xacro:sick_tim310 name="laser" ros_topic="scan" />
+  <xacro:include filename="$(find ur5_manipulation)/urdf/ur5.urdf.xacro" />
   <!-- arm -->
   <xacro:ur5_robot prefix="" joint_limited="false"/>
@@ -11,11 +9,6 @@
   <joint name="world_joint" type="fixed">
     <parent link="world" />
-    <child link = "base_link" />
+    <child link = "ur5_base_link" />
     <origin xyz="0.0 0.0 0.75" rpy="0.0 0.0 0.0" />
   </joint>
-  <joint name="tim_link" type="fixed">
-	<parent link="base_link" />
-    <child link = "laser_mount_link" />
-    <origin xyz="-0.28 0.01 0" rpy="0.0 0.0 3.142" />
-  </joint>
 </robot>
